Commit message: add support to /odom

File: src/launch/basestation_launch/urdf/f1tenth_ucsd.urdf (robot description, URDF)
Before this commit: robot my_robot, 8 links, 7 joints
Links:
- link base_link: geometry collision cylinder length=0.09 radius=0.06; visual box size=0.20 0.5 0.05
- link camera_link: geometry visual box size=0.097 0.03 0.023
- link lidar_link: geometry visual box size=0.065 0.065 0.06
- link wheel_FL: geometry visual cylinder length=0.045 radius=0.05
- link wheel_FR: geometry visual cylinder length=0.045 radius=0.05
- link wheel_RL: geometry visual cylinder length=0.045 radius=0.05
- link wheel_RR: geometry visual cylinder length=0.045 radius=0.05
Joints:
- joint base_footprint_joint: origin xyz=0 0 0 rpy=0 0 0 -> xyz=0 0 -0.05 rpy=0 0 0
- joint camera_joint: parent lidar_link -> base_link

Commit message: urdf fixed

File: src/launch/basestation_launch/urdf/f1tenth_ucsd.urdf (robot description, URDF)
Before this commit: robot my_robot, 8 links, 7 joints
Joints:
- joint camera_joint: origin xyz=0.0 0.0 0.0 rpy=0 0 0 -> xyz=0.120 0.0 0.145 rpy=0 0 0
- joint lidar_joint: origin xyz=0.0 0.0 0.0 rpy=0 0 0 -> xyz=0.01 0.0 0.20 rpy=0 0 0
- joint wheel_FL_joint: origin xyz=0.0 0.0 0.0 rpy=0 0 0 -> xyz=0.160 0.120 0.0 rpy=0 0 0
- joint wheel_FR_joint: origin xyz=0.0 0.0 0.0 rpy=0 0 0 -> xyz=0.160 -0.120 0.0 rpy=0 0 0
- joint wheel_RL_joint: origin xyz=0.0 0.0 0.0 rpy=0 0 0 -> xyz=-0.160 0.120 0.0 rpy=0 0 0
- joint wheel_RR_joint: origin xyz=0.0 0.0 0.0 rpy=0 0 0 -> xyz=-0.160 -0.120 0.0 rpy=0 0 0

Commit message: minor fix, starts working on ekf

File: src/launch/basestation_launch/urdf/f1tenth_ucsd.urdf (robot description, URDF)
Before this commit: robot my_robot, 8 links, 7 joints
Joints:
- joint base_footprint_joint: child base_footprint -> base_link; origin xyz=0 0 -0.05 rpy=0 0 0 -> xyz=0 0 0.05 rpy=0 0 0; parent base_link -> base_footprint
