Commit message: update urdf file, add `ego_racecar/` as prefix every frame, except `odom`, `map`, and frames from sensors themselves

File: src/launch/basestation_launch/urdf/ucsd_racecar.xacro (robot description, xacro)
@@ -7,5 +7,5 @@
     <xacro:property name="wheel_radius" value="0.0508" />
     <xacro:property name="wheel_length" value="0.0381" />
-    <xacro:property name="laser_distance_from_base_link" value="0.275" />
+    <!-- <xacro:property name="laser_distance_from_base_link" value="0.275" /> -->
     <!-- <xacro:property name="laser_height" value="0.05" /> -->
     <!-- <xacro:property name="laser_radius" value="0.026" /> -->
@@ -24,5 +24,5 @@
     </material>
     <!-- BASE LINK -->
-    <link name="base_link">
+    <link name="${car_name}/base_link">
         <inertial>
             <origin xyz="0 0 0.05" rpy="0 0 0"/>
@@ -45,13 +45,13 @@
     </link>
     <!-- BASE FOOTPRINT LINK-->
-    <link name="base_footprint">
+    <link name="${car_name}/base_footprint">
     </link>
     <joint name="base_footprint_joint" type="fixed">
-        <parent link="base_footprint"/>
-        <child link="base_link"/>
+        <parent link="${car_name}/base_footprint"/>
+        <child link="${car_name}/base_link"/>
         <origin xyz="0 0 ${wheel_radius}" rpy="0 0 0"/>
     </joint>
     <!-- LIDAR LINK -->
-    <link name="lidar_link">
+    <link name="${car_name}/lidar_link">
 	<visual>
             <origin rpy="0 0 ${pi/2}" xyz="0.0 0.0 0.0"/>
@@ -63,10 +63,10 @@
     </link>
     <joint name="lidar_joint" type="fixed">
-        <parent link="base_link"/>
-        <child link="lidar_link"/>
+        <parent link="${car_name}/base_link"/>
+        <child link="${car_name}/lidar_link"/>
         <origin xyz="0.05 0.0 0.10" rpy="0 0 0"/>
     </joint>
     <!-- CAMERA LINK -->
-    <link name="camera_link">
+    <link name="${car_name}/camera_link">
 	    <visual>
             <origin rpy="0 0 ${pi/2}" xyz="0.0 0.0 0.0"/>
@@ -78,6 +78,6 @@
     </link>
     <joint name="camera_joint" type="fixed">
-        <parent link="base_link"/>
-        <child link="camera_link"/>
+        <parent link="${car_name}/base_link"/>
+        <child link="${car_name}/camera_link"/>
         <origin xyz="0.120 0.0 0.145" rpy="0 0 0"/>
     </joint>
@@ -94,5 +94,5 @@
     <link name="${car_name}/hinge_FL"/>
     <joint name="base_to_hinge_FL" type="fixed">
-        <parent link="base_link"/>
+        <parent link="${car_name}/base_link"/>
         <child link="${car_name}/hinge_FL"/>
         <origin xyz="${wheelbase/2} ${(wheel_length+width)/2} 0.0" rpy="0 0 0"/>
@@ -116,5 +116,5 @@
     <link name="${car_name}/hinge_FR"/>
     <joint name="base_to_hinge_FR" type="fixed">
-        <parent link="base_link"/>
+        <parent link="${car_name}/base_link"/>
         <child link="${car_name}/hinge_FR"/>
         <origin xyz="${wheelbase/2} -${(wheel_length+width)/2} 0.0" rpy="0 0 0"/>
@@ -137,5 +137,5 @@
     </link>
     <joint name="wheel_RL_joint" type="revolute">
-        <parent link="base_link"/>
+        <parent link="${car_name}/base_link"/>
         <child link="${car_name}/wheel_RL"/>
         <origin xyz="-${wheelbase/2} ${(wheel_length+width)/2} 0.0" rpy="0 0 0"/>
@@ -154,5 +154,5 @@
     </link>
     <joint name="wheel_RR_joint" type="revolute">
-        <parent link="base_link"/>
+        <parent link="${car_name}/base_link"/>
         <child link="${car_name}/wheel_RR"/>
         <origin xyz="-${wheelbase/2} -${(wheel_length+width)/2} 0.0" rpy="0 0 0"/>
@@ -161,5 +161,5 @@
     </joint>
     <!-- GAZEBO -->
-    <gazebo reference="base_link">
+    <gazebo reference="${car_name}/base_link">
         <kp>100000.0</kp>
         <kd>100000.0</kd>
@@ -169,5 +169,5 @@
     </gazebo>
     <!-- camera -->
-    <gazebo reference="camera_link">
+    <gazebo reference="${car_name}/camera_link">
         <sensor type="camera" name="camera1">
         <update_rate>15.0</update_rate>
@@ -195,5 +195,5 @@
             <imageTopicName>image_raw</imageTopicName>
             <cameraInfoTopicName>camera_info</cameraInfoTopicName>
-            <frameName>camera_link</frameName>
+            <frameName>${car_name}/camera_link</frameName>
             <hackBaseline>0.07</hackBaseline>
             <distortionK1>0.0</distortionK1>
@@ -205,5 +205,5 @@
         </sensor>
     </gazebo>
-    <gazebo reference="lidar_link">
+    <gazebo reference="${car_name}/lidar_link">
         <material value="Gazebo/Blue" />
         <sensor type="ray" name="lidar">
@@ -229,5 +229,5 @@
             <plugin name="scan" filename="libgazebo_ros_gpu_laser.so">
             <topicName>/ego_racecar/scan</topicName>
-            <frameName>lidar_link</frameName>
+            <frameName>${car_name}/lidar_link</frameName>
             </plugin>
         </sensor>
