Commit message: [Feat] modified autodrive_racecar.xacro to given spec

File: src/launch/basestation_launch/urdf/autodrive_racecar.xacro (robot description, xacro)
@@ -1,10 +1,10 @@
 <?xml version="1.0"?>
 <robot xmlns:xacro="http://www.ros.org/wiki/xacro" name="racecar">
-    <xacro:property name="wheelbase" value="0.3302" />
-    <xacro:property name="width" value="0.2032" />
+    <xacro:property name="wheelbase" value="0.3240" />
+    <xacro:property name="width" value="0.1800" />
     <xacro:property name="height" value="0.05" />
     <!-- <xacro:property name="ground_offset" value="0.04" /> -->
-    <xacro:property name="wheel_radius" value="0.0508" />
-    <xacro:property name="wheel_length" value="0.0381" />
+    <xacro:property name="wheel_radius" value="0.0590" />
+    <xacro:property name="wheel_length" value="0.0450" />
     <!-- <xacro:property name="laser_distance_from_base_link" value="0.275" /> -->
     <!-- <xacro:property name="laser_height" value="0.05" /> -->
@@ -65,5 +65,5 @@
         <parent link="${car_name}/base_link"/>
         <child link="${car_name}/lidar_link"/>
-        <origin xyz="0.05 0.0 0.10" rpy="0 0 0"/>
+        <origin xyz="${0.2733 - wheelbase/2} 0.0 0.096" rpy="0 0 0"/>
     </joint>
     <!-- CAMERA LINK -->
@@ -74,11 +74,26 @@
                 <box size="0.097 0.03 0.023"/>
             </geometry>
+            <material name="black"/>
+        </visual>
+    </link>
+    <joint name="camera_joint" type="fixed">
+        <parent link="${car_name}/base_link"/>
+        <child link="${car_name}/camera_link"/>
+        <origin xyz="${-0.015 - wheelbase/2} 0.0 0.15" rpy="0 ${10*pi/180} 0"/>
+    </joint>
+    <!-- IMU LINK -->
+    <link name="${car_name}/imu_link">
+	    <visual>
+            <origin rpy="0 0 ${pi/2}" xyz="0.0 0.0 0.0"/>
+            <geometry>
+                <box size="0.03 0.03 0.003"/>
+            </geometry>
             <material name="grey"/>
         </visual>
     </link>
-    <joint name="camera_joint" type="fixed">
-        <parent link="${car_name}/base_link"/>
-        <child link="${car_name}/camera_link"/>
-        <origin xyz="0.120 0.0 0.145" rpy="0 0 0"/>
+    <joint name="imu_joint" type="fixed">
+        <parent link="${car_name}/base_link"/>
+        <child link="${car_name}/imu_link"/>
+        <origin xyz="${0.08 - wheelbase/2} 0.0 0.055" rpy="0 0 0"/>
     </joint>
     <!-- WHEEL FL LINK -->

Commit message: [Refactor] front wheels joint type changes to `continuous`

File: src/launch/basestation_launch/urdf/autodrive_racecar.xacro (robot description, xacro)
@@ -113,5 +113,5 @@
         <origin xyz="${wheelbase/2} ${(wheel_length+width)/2} 0.0" rpy="0 0 0"/>
     </joint>
-    <joint name="wheel_FL_joint" type="revolute">
+    <joint name="wheel_FL_joint" type="continuous">
         <parent link="${car_name}/hinge_FL"/>
         <child link="${car_name}/wheel_FL"/>
@@ -135,5 +135,5 @@
         <origin xyz="${wheelbase/2} -${(wheel_length+width)/2} 0.0" rpy="0 0 0"/>
     </joint>
-    <joint name="wheel_FR_joint" type="revolute">
+    <joint name="wheel_FR_joint" type="continuous">
         <parent link="${car_name}/hinge_FR"/>
         <child link="${car_name}/wheel_FR"/>
