Commit message: fix typo

File: src/common/common_metadata/urdf/robocar/robocar.urdf (robot description, URDF)
Before this commit: robot AV 21, 40 links, 39 joints
Links:
- link model: geometry visual mesh filename=package://common_metadata/urdf/iac_car/visual/il15_body.stl scale=0.01 0.01 0.01
- link tyre_fl: geometry visual mesh filename=package://common_metadata/urdf/iac_car/visual/il15_tyre_fl.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 scale=0.01 0.01 0.01
- link tyre_fr: geometry visual mesh filename=package://common_metadata/urdf/iac_car/visual/il15_tyre_fr.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 scale=0.01 0.01 0.01
- link tyre_rl: geometry visual mesh filename=package://common_metadata/urdf/iac_car/visual/il15_tyre_rl.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 scale=0.01 0.01 0.01
- link tyre_rr: geometry visual mesh filename=package://common_metadata/urdf/iac_car/visual/il15_tyre_rr.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 scale=0.01 0.01 0.01

Commit message: add autonomy_launch

File: src/common/common_metadata/urdf/robocar/robocar.urdf (robot description, URDF)
Before this commit: robot AV 21, 40 links, 39 joints
Links:
- removed link camera_left
- removed link camera_rear
- removed link camera_right
- removed link gps_antenna_left
- removed link gps_antenna_rear
- removed link gps_antenna_right
- removed link gps_bottom
- removed link imu_bottom
- removed link imu_vectornav
- removed link luminar_front
- removed link luminar_left
- removed link luminar_rear
- removed link luminar_right
- removed link radar_front
- removed link radar_rear
- removed link vectornav
- removed link vimba_front
- removed link vimba_front_left_center
- removed link vimba_front_right_center
- removed link vimba_left
- removed link vimba_rear
- removed link vimba_right
- added link livox_front
- link model: geometry visual mesh filename=package://common_metadata/urdf/robocar/visual/il15_body.stl scale=0.01 0.01 0.01
- link tyre_fl: geometry visual mesh filename=package://common_metadata/urdf/robocar/visual/il15_tyre_fl.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 scale=0.01 0.01 0.01
- link tyre_fr: geometry visual mesh filename=package://common_metadata/urdf/robocar/visual/il15_tyre_fr.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 scale=0.01 0.01 0.01
- link tyre_rl: geometry visual mesh filename=package://common_metadata/urdf/robocar/visual/il15_tyre_rl.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 scale=0.01 0.01 0.01
- link tyre_rr: geometry visual mesh filename=package://common_metadata/urdf/robocar/visual/il15_tyre_rr.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 scale=0.01 0.01 0.01
Joints:
- removed joint camera_left_joint
- removed joint camera_rear_joint
- removed joint camera_right_joint
- removed joint gps_antenna_left_joint
- removed joint gps_antenna_rear_joint
- removed joint gps_antenna_right_joint
- removed joint gps_bottom_joint
- removed joint imu_bottom_joint
- removed joint imu_vectornav_joint
- removed joint luminar_front_joint
- removed joint luminar_left_joint
- removed joint luminar_rear_joint
- removed joint luminar_right_joint
- removed joint radar_front_joint
- removed joint radar_rear_joint
- removed joint vectornav_joint
- removed joint vimba_front_joint
- removed joint vimba_front_left_center_joint
- removed joint vimba_front_right_center_joint
- removed joint vimba_left_joint
- removed joint vimba_rear_joint
- removed joint vimba_right_joint
- added joint livox_front_joint: type fixed, parent base_link, child livox_front, origin xyz=2.22177 0.00541 0.46683 rpy=0.0 0.0 0.0
- joint cg_joint: origin xyz=1.248 0.0 0.077 -> xyz=${(wheelbase_rear-wheelbase_front)/2} 0.0 0.074
- joint wheel_base: origin xyz=2.9729 0.0 0.0 -> xyz=${(wheelbase_front+wheelbase_rear)/2} 0.0 0.0
